Commit message: (feat)添加依赖，编译成功

File: ros2_ws/install/panda_moveit_config/share/panda_moveit_config/config/panda.ros2_control.xacro (robot description, xacro)
@@ -1,68 +1 @@
-<?xml version="1.0"?>
-<robot xmlns:xacro="http://www.ros.org/wiki/xacro">
-    <xacro:macro name="panda_ros2_control" params="name initial_positions_file">
-        <xacro:property name="initial_positions" value="${load_yaml(initial_positions_file)['initial_positions']}"/>
-        <ros2_control name="${name}" type="system">
-            <hardware>
-                <!-- By default, set up controllers for simulation. This won't work on real hardware -->
-                <plugin>mock_components/GenericSystem</plugin>
-            </hardware>
-            <joint name="panda_joint1">
-                <command_interface name="position"/>
-                <state_interface name="position">
-                  <param name="initial_value">${initial_positions['panda_joint1']}</param>
-                </state_interface>
-                <state_interface name="velocity"/>
-            </joint>
-            <joint name="panda_joint2">
-                <command_interface name="position"/>
-                <state_interface name="position">
-                  <param name="initial_value">${initial_positions['panda_joint2']}</param>
-                </state_interface>
-                <state_interface name="velocity"/>
-            </joint>
-            <joint name="panda_joint3">
-                <command_interface name="position"/>
-                <state_interface name="position">
-                  <param name="initial_value">${initial_positions['panda_joint3']}</param>
-                </state_interface>
-                <state_interface name="velocity"/>
-            </joint>
-            <joint name="panda_joint4">
-                <command_interface name="position"/>
-                <state_interface name="position">
-                  <param name="initial_value">${initial_positions['panda_joint4']}</param>
-                </state_interface>
-                <state_interface name="velocity"/>
-            </joint>
-            <joint name="panda_joint5">
-                <command_interface name="position"/>
-                <state_interface name="position">
-                  <param name="initial_value">${initial_positions['panda_joint5']}</param>
-                </state_interface>
-                <state_interface name="velocity"/>
-            </joint>
-            <joint name="panda_joint6">
-                <command_interface name="position"/>
-                <state_interface name="position">
-                  <param name="initial_value">${initial_positions['panda_joint6']}</param>
-                </state_interface>
-                <state_interface name="velocity"/>
-            </joint>
-            <joint name="panda_joint7">
-                <command_interface name="position"/>
-                <state_interface name="position">
-                  <param name="initial_value">${initial_positions['panda_joint7']}</param>
-                </state_interface>
-                <state_interface name="velocity"/>
-            </joint>
-            <joint name="panda_finger_joint1">
-                <command_interface name="position"/>
-                <state_interface name="position">
-                  <param name="initial_value">${initial_positions['panda_finger_joint1']}</param>
-                </state_interface>
-                <state_interface name="velocity"/>
-            </joint>
-        </ros2_control>
-    </xacro:macro>
-</robot>
+/home/yc-dlan/Dlancy_moveit2/ros2_ws/src/moveit_resources/panda_moveit_config/config/panda.ros2_control.xacro

File: ros2_ws/install/panda_moveit_config/share/panda_moveit_config/config/panda.urdf.xacro (robot description, xacro)
@@ -1,9 +1 @@
-<?xml version="1.0"?>
-<robot xmlns:xacro="http://www.ros.org/wiki/xacro" name="panda">
-    <xacro:arg name="initial_positions_file" default="initial_positions.yaml" />
-    <!-- Import panda urdf file -->
-    <xacro:include filename="$(find my_moveit2driver)/urdf/panda.urdf" />
-    <!-- Import control_xacro -->
-    <xacro:include filename="panda.ros2_control.xacro" />
-    <xacro:panda_ros2_control name="FakeSystem" initial_positions_file="$(arg initial_positions_file)"/>
-</robot>
+/home/yc-dlan/Dlancy_moveit2/ros2_ws/src/moveit_resources/panda_moveit_config/config/panda.urdf.xacro
